File: msxrom.sch (EAGLE design)
At the start: 15 parts, among them X2 2526-

Commit message: loose files
Connections:
- removed net !IOSEL: V21.Y, X2-7.KL
- new net IOSEL: V21.W, X2-7.KL
- net !RESET: now also JP1.!RESET
Changed lines of the file:
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@@
 <wire x1="-7.62" y1="127" x2="-12.7" y2="127" width="0.1524" layer="91"/>
 <junction x="-7.62" y="127"/>
-<label x="63.5" y="99.06" size="1.778" layer="95"/>
+<label x="-15.24" y="127" size="1.778" layer="95"/>
 </segment>
 <segment>
@@
 </segment>
 </net>
-<net name="!IOSEL" class="0">
-<segment>
-<pinref part="V2" gate="1" pin="Y"/>
-<wire x1="99.06" y1="152.4" x2="111.76" y2="152.4" width="0.1524" layer="91"/>
-<label x="109.22" y="152.4" size="1.778" layer="95"/>
+<net name="D0" class="0">
+<segment>
+<wire x1="223.52" y1="160.02" x2="205.74" y2="160.02" width="0.1524" layer="91"/>
+<label x="223.52" y="160.02" size="1.778" layer="95" font="vector" xref="yes"/>
+<pinref part="X2" gate="-23" pin="KL"/>
+</segment>
+<segment>
+<pinref part="JP1" gate="CRTRDG" pin="D0"/>
+<pinref part="IC1" gate="G$1" pin="O0"/>
+<wire x1="-7.62" y1="86.36" x2="29.21" y2="86.36" width="0.1524" layer="91"/>
+</segment>
+</net>
+<net name="D1" class="0">
+<segment>
+<wire x1="210.82" y1="157.48" x2="205.74" y2="157.48" width="0.1524" layer="91"/>
+<label x="210.82" y="157.48" size="1.778" layer="95" font="vector" xref="yes"/>
+<pinref part="X2" gate="-21" pin="KL"/>
+</segment>
+<segment>
+<pinref part="JP1" gate="CRTRDG" pin="D1"/>
+<pinref part="IC1" gate="G$1" pin="O1"/>
+<wire x1="-7.62" y1="83.82" x2="29.21" y2="83.82" width="0.1524" layer="91"/>
+</segment>
+</net>
+<net name="D2" class="0">
+<segment>
+<wire x1="223.52" y1="154.94" x2="205.74" y2="154.94" width="0.1524" layer="91"/>
+<label x="223.52" y="154.94" size="1.778" layer="95" font="vector" xref="yes"/>
+<pinref part="X2" gate="-19" pin="KL"/>
+</segment>
+<segment>
+<pinref part="JP1" gate="CRTRDG" pin="D2"/>
+<pinref part="IC1" gate="G$1" pin="O2"/>
+<wire x1="-7.62" y1="81.28" x2="29.21" y2="81.28" width="0.1524" layer="91"/>
+</segment>
+</net>
+<net name="D5" class="0">
+<segment>
+<label x="210.82" y="147.32" size="1.778" layer="95" font="vector" xref="yes"/>
+<wire x1="210.82" y1="147.32" x2="205.74" y2="147.32" width="0.1524" layer="91"/>
+<pinref part="X2" gate="-13" pin="KL"/>
+</segment>
+<segment>
+<pinref part="JP1" gate="CRTRDG" pin="D5"/>
+<pinref part="IC1" gate="G$1" pin="O5"/>
+<wire x1="-7.62" y1="73.66" x2="29.21" y2="73.66" width="0.1524" layer="91"/>
+</segment>
+</net>
+<net name="D7" class="0">
+<segment>
+<label x="210.82" y="142.24" size="1.778" layer="95" font="vector" xref="yes"/>
+<wire x1="210.82" y1="142.24" x2="205.74" y2="142.24" width="0.1524" layer="91"/>
+<pinref part="X2" gate="-9" pin="KL"/>
+</segment>
+<segment>
+<pinref part="JP1" gate="CRTRDG" pin="D7"/>
+<pinref part="IC1" gate="G$1" pin="O7"/>
+<wire x1="-7.62" y1="68.58" x2="29.21" y2="68.58" width="0.1524" layer="91"/>
+</segment>
+</net>
+<net name="!RESET" class="0">
+<segment>
+<wire x1="180.34" y1="139.7" x2="193.04" y2="139.7" width="0.1524" layer="91"/>
+<label x="180.34" y="139.7" size="1.778" layer="95" font="vector" rot="R180" xref="yes"/>
+<pinref part="X2" gate="-8" pin="KL"/>
+</segment>
+<segment>
+<pinref part="JP1" gate="CRTRDG" pin="!RESET"/>
+<wire x1="45.72" y1="55.88" x2="29.21" y2="55.88" width="0.1524" layer="91"/>
+<label x="40.64" y="55.88" size="1.778" layer="95"/>
+</segment>
+</net>
+<net name="D3" class="0">
+<segment>
+<wire x1="210.82" y1="152.4" x2="205.74" y2="152.4" width="0.1524" layer="91"/>
+<label x="210.82" y="152.4" size="1.778" layer="95" font="vector" xref="yes"/>
+<pinref part="X2" gate="-17" pin="KL"/>
+</segment>
+<segment>
+<pinref part="JP1" gate="CRTRDG" pin="D3"/>
+<pinref part="IC1" gate="G$1" pin="O3"/>
+<wire x1="-7.62" y1="78.74" x2="29.21" y2="78.74" width="0.1524" layer="91"/>
+</segment>
+</net>
+<net name="D4" class="0">
+<segment>
+<label x="223.52" y="149.86" size="1.778" layer="95" font="vector" xref="yes"/>
+<wire x1="223.52" y1="149.86" x2="205.74" y2="149.86" width="0.1524" layer="91"/>
+<pinref part="X2" gate="-15" pin="KL"/>
+</segment>
+<segment>
+<pinref part="JP1" gate="CRTRDG" pin="D4"/>
+<pinref part="IC1" gate="G$1" pin="O4"/>
+<wire x1="-7.62" y1="76.2" x2="29.21" y2="76.2" width="0.1524" layer="91"/>
+</segment>
+</net>
+<net name="D6" class="0">
+<segment>
+<wire x1="223.52" y1="144.78" x2="205.74" y2="144.78" width="0.1524" layer="91"/>
+<label x="223.52" y="144.78" size="1.778" layer="95" font="vector" xref="yes"/>
+<pinref part="X2" gate="-11" pin="KL"/>
+</segment>
+<segment>
+<pinref part="JP1" gate="CRTRDG" pin="D6"/>
+<pinref part="IC1" gate="G$1" pin="O6"/>
+<wire x1="-7.62" y1="71.12" x2="29.21" y2="71.12" width="0.1524" layer="91"/>
+</segment>
+</net>
+<net name="TX-S" class="0">
+<segment>
+<label x="185.42" y="132.08" size="1.778" layer="95" font="vector" rot="R180" xref="yes"/>
+<pinref part="X2" gate="-2" pin="KL"/>
+<wire x1="193.04" y1="132.08" x2="185.42" y2="132.08" width="0.1524" layer="91"/>
+</segment>
+</net>
+<net name="RX-S" class="0">
+<segment>
+<label x="175.26" y="134.62" size="1.778" layer="95" rot="R180" xref="yes"/>
+<pinref part="X2" gate="-4" pin="KL"/>
+<wire x1="193.04" y1="134.62" x2="175.26" y2="134.62" width="0.1524" layer="91"/>
+</segment>
+</net>
+<net name="IOSEL" class="0">
+<segment>
+<wire x1="99.06" y1="127" x2="111.76" y2="127" width="0.1524" layer="91"/>
+<pinref part="V2" gate="1" pin="W"/>
+<label x="106.68" y="127" size="1.778" layer="95"/>
 </segment>
 <segment>
@@
 </segment>
 </net>
-<net name="D0" class="0">
-<segment>
-<wire x1="223.52" y1="160.02" x2="205.74" y2="160.02" width="0.1524" layer="91"/>
-<label x="223.52" y="160.02" size="1.778" layer="95" font="vector" xref="yes"/>
-<pinref part="X2" gate="-23" pin="KL"/>
-</segment>
-<segment>
-<pinref part="JP1" gate="CRTRDG" pin="D0"/>
-<pinref part="IC1" gate="G$1" pin="O0"/>
-<wire x1="-7.62" y1="86.36" x2="29.21" y2="86.36" width="0.1524" layer="91"/>
-</segment>
-</net>
-<net name="D1" class="0">
-<segment>
-<wire x1="210.82" y1="157.48" x2="205.74" y2="157.48" width="0.1524" layer="91"/>
-<label x="210.82" y="157.48" size="1.778" layer="95" font="vector" xref="yes"/>
-<pinref part="X2" gate="-21" pin="KL"/>
-</segment>
-<segment>
-<pinref part="JP1" gate="CRTRDG" pin="D1"/>
-<pinref part="IC1" gate="G$1" pin="O1"/>
-<wire x1="-7.62" y1="83.82" x2="29.21" y2="83.82" width="0.1524" layer="91"/>
-</segment>
-</net>
-<net name="D2" class="0">
-<segment>
-<wire x1="223.52" y1="154.94" x2="205.74" y2="154.94" width="0.1524" layer="91"/>
-<label x="223.52" y="154.94" size="1.778" layer="95" font="vector" xref="yes"/>
-<pinref part="X2" gate="-19" pin="KL"/>
-</segment>
-<segment>
-<pinref part="JP1" gate="CRTRDG" pin="D2"/>
-<pinref part="IC1" gate="G$1" pin="O2"/>
-<wire x1="-7.62" y1="81.28" x2="29.21" y2="81.28" width="0.1524" layer="91"/>
-</segment>
-</net>
-<net name="D5" class="0">
-<segment>
-<label x="210.82" y="147.32" size="1.778" layer="95" font="vector" xref="yes"/>
-<wire x1="210.82" y1="147.32" x2="205.74" y2="147.32" width="0.1524" layer="91"/>
-<pinref part="X2" gate="-13" pin="KL"/>
-</segment>
-<segment>
-<pinref part="JP1" gate="CRTRDG" pin="D5"/>
-<pinref part="IC1" gate="G$1" pin="O5"/>
-<wire x1="-7.62" y1="73.66" x2="29.21" y2="73.66" width="0.1524" layer="91"/>
-</segment>
-</net>
-<net name="D7" class="0">
-<segment>
-<label x="210.82" y="142.24" size="1.778" layer="95" font="vector" xref="yes"/>
-<wire x1="210.82" y1="142.24" x2="205.74" y2="142.24" width="0.1524" layer="91"/>
-<pinref part="X2" gate="-9" pin="KL"/>
-</segment>
-<segment>
-<pinref part="JP1" gate="CRTRDG" pin="D7"/>
-<pinref part="IC1" gate="G$1" pin="O7"/>
-<wire x1="-7.62" y1="68.58" x2="29.21" y2="68.58" width="0.1524" layer="91"/>
-</segment>
-</net>
-<net name="!RESET" class="0">
-<segment>
-<wire x1="180.34" y1="139.7" x2="193.04" y2="139.7" width="0.1524" layer="91"/>
-<label x="180.34" y="139.7" size="1.778" layer="95" font="vector" rot="R180" xref="yes"/>
-<pinref part="X2" gate="-8" pin="KL"/>
-</segment>
-</net>
-<net name="D3" class="0">
-<segment>
-<wire x1="210.82" y1="152.4" x2="205.74" y2="152.4" width="0.1524" layer="91"/>
-<label x="210.82" y="152.4" size="1.778" layer="95" font="vector" xref="yes"/>
-<pinref part="X2" gate="-17" pin="KL"/>
-</segment>
-<segment>
-<pinref part="JP1" gate="CRTRDG" pin="D3"/>
-<pinref part="IC1" gate="G$1" pin="O3"/>
-<wire x1="-7.62" y1="78.74" x2="29.21" y2="78.74" width="0.1524" layer="91"/>
-</segment>
-</net>
-<net name="D4" class="0">
-<segment>
-<label x="223.52" y="149.86" size="1.778" layer="95" font="vector" xref="yes"/>
-<wire x1="223.52" y1="149.86" x2="205.74" y2="149.86" width="0.1524" layer="91"/>
-<pinref part="X2" gate="-15" pin="KL"/>
-</segment>
-<segment>
-<pinref part="JP1" gate="CRTRDG" pin="D4"/>
-<pinref part="IC1" gate="G$1" pin="O4"/>
-<wire x1="-7.62" y1="76.2" x2="29.21" y2="76.2" width="0.1524" layer="91"/>
-</segment>
-</net>
-<net name="D6" class="0">
-<segment>
-<wire x1="223.52" y1="144.78" x2="205.74" y2="144.78" width="0.1524" layer="91"/>
-<label x="223.52" y="144.78" size="1.778" layer="95" font="vector" xref="yes"/>
-<pinref part="X2" gate="-11" pin="KL"/>
-</segment>
-<segment>
-<pinref part="JP1" gate="CRTRDG" pin="D6"/>
-<pinref part="IC1" gate="G$1" pin="O6"/>
-<wire x1="-7.62" y1="71.12" x2="29.21" y2="71.12" width="0.1524" layer="91"/>
-</segment>
-</net>
-<net name="TX-S" class="0">
-<segment>
-<label x="185.42" y="132.08" size="1.778" layer="95" font="vector" rot="R180" xref="yes"/>
-<pinref part="X2" gate="-2" pin="KL"/>
-<wire x1="193.04" y1="132.08" x2="185.42" y2="132.08" width="0.1524" layer="91"/>
-</segment>
-</net>
-<net name="RX-S" class="0">
-<segment>
-<label x="175.26" y="134.62" size="1.778" layer="95" rot="R180" xref="yes"/>
-<pinref part="X2" gate="-4" pin="KL"/>
-<wire x1="193.04" y1="134.62" x2="175.26" y2="134.62" width="0.1524" layer="91"/>
-</segment>
-</net>
