File: esmsx.brd (EAGLE design)
At the start: 92.7 x 63.5 mm, 43 parts, among them IC2 317EMP

Commit message: led section and renaming signal
Connections:
- net LED-BLUE renamed !LED-BLUE
Changed lines of the file:
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@@
 <wire x1="3.96875" y1="46.83125" x2="3.4925" y2="46.83125" width="0.254" layer="16"/>
 </signal>
-<signal name="LED-BLUE">
+<signal name="!LED-BLUE">
 <contactref element="PIC32MX150F128D" pad="24"/>
 <wire x1="9.642703125" y1="49.331246875" x2="8.7744" y2="50.19955" width="0.254" layer="16"/>
